Commit message: Added box inertia tags for camera in my_robot.xacro

File: Project2/src/my_robot/urdf/my_robot.xacro (robot description, xacro)
@@ -105,5 +105,5 @@
     <inertial>
       <mass value="0.1"/>
-      <origin xyz="0.05 0.05 0.05" rpy=" 0 0 0"/>
+      <origin xyz="0 0 0" rpy=" 0 0 0"/>
       <inertia
           ixx="1e-6" ixy="0" ixz="0"
@@ -124,4 +124,7 @@
       </geometry>
     </visual>
+    <box_inertia sizeX="0.05" sizeY="0.05" sizeZ="0.05" mass="0.1">
+      <origin xyz="0 0 0" rpy="0 0 0" />
+    </box_inertia>
   </link>
   <link name='hokuyo'>

Commit message: Customized robot appearance

File: Project2/src/my_robot/urdf/my_robot.xacro (robot description, xacro)
@@ -1,3 +1,5 @@
 <?xml version='1.0'?>
+<!-- Per the bug described here: https://bitbucket.org/osrf/sdformat/issues/132/parser-does-not-handle-urdf-material, the name attribute was removed from tags.
+This allows colors to be applied to the links -->
 <robot name="my_robot" xmlns:xacro="http://www.ros.org/wiki/xacro">
   <xacro:include filename="$(find my_robot)/urdf/my_robot.gazebo" />
@@ -19,16 +21,74 @@
       />
     </inertial>
-    <collision name='collision'>
-      <origin xyz="0 0 0" rpy=" 0 0 0"/>
-      <geometry>
-        <box size=".4 .2 .1"/>
-      </geometry>
-    </collision>
-    <visual name='chassis_visual'>
-      <origin xyz="0 0 0" rpy=" 0 0 0"/>
-      <geometry>
-        <box size=".4 .2 .1"/>
-      </geometry>
-    </visual>
+    <collision name='chassis_bottom'>
+      <origin xyz="0 0 0" rpy=" 0 0 0"/>
+      <geometry>
+        <box size=".4 .3 .05"/>
+      </geometry>
+    </collision>
+    <!--  name='chassis_bottom_visual' -->
+    <visual>
+      <origin xyz="0 0 0" rpy=" 0 0 0"/>
+      <geometry>
+        <box size=".4 .3 .05"/>
+      </geometry>
+    </visual>
+    <collision name='chassis_top'>
+      <origin xyz="0 0 0.2" rpy=" 0 0 0"/>
+      <geometry>
+        <box size=".4 .3 .05"/>
+      </geometry>
+    </collision>
+    <!--  name='chassis_top_visual' -->
+    <visual>
+      <origin xyz="0 0 0.2" rpy=" 0 0 0"/>
+      <geometry>
+        <box size=".4 .3 .05"/>
+      </geometry>
+    </visual>
+    <!-- Support posts -->
+    <!--  name='post_FL_visual' -->
+    <visual>
+      <origin xyz="0.18 0.13 0.1" rpy=" 0 0 0"/>
+      <geometry>
+        <cylinder length="0.2" radius="0.01"/>
+      </geometry>
+    </visual>
+    <!--  name='post_FR_visual' -->
+    <visual>
+      <origin xyz="0.18 -0.13 0.1" rpy=" 0 0 0"/>
+      <geometry>
+        <cylinder length="0.2" radius="0.01"/>
+      </geometry>
+    </visual>
+    <!--  name='post_BL_visual' -->
+    <visual>
+      <origin xyz="-0.18 0.13 0.1" rpy=" 0 0 0"/>
+      <geometry>
+        <cylinder length="0.2" radius="0.01"/>
+      </geometry>
+    </visual>
+    <!--  name='post_BR_visual' -->
+    <visual>
+      <origin xyz="-0.18 -0.13 0.1" rpy=" 0 0 0"/>
+      <geometry>
+        <cylinder length="0.2" radius="0.01"/>
+      </geometry>
+    </visual>
+    <collision name='posts_collision'>
+      <origin xyz="0 0 0.1" rpy=" 0 0 0"/>
+      <geometry>
+        <box size=".4 .3 .2"/>
+      </geometry>
+    </collision>
+    <!-- camera mount -->
+    <!--  name='camera_mount_visual' -->
+    <visual>
+      <origin xyz="0.17 0 0.055" rpy=" 0 0 0"/>
+      <geometry>
+        <box size=".01 .06 .06"/>
+      </geometry>
+    </visual>
+    <!-- casters -->
     <collision name='back_caster_collision'>
       <origin xyz="-0.15 0 -0.05" rpy=" 0 0 0"/>
@@ -37,4 +97,5 @@
       </geometry>
     </collision>
+    <!--  name='back_caster_visual' -->
     <visual name='back_caster_visual'>
       <origin xyz="-0.15 0 -0.05" rpy=" 0 0 0"/>
@@ -49,4 +110,5 @@
       </geometry>
     </collision>
+    <!--  name='front_caster_visual' -->
     <visual name='front_caster_visual'>
       <origin xyz="0.15 0 -0.05" rpy=" 0 0 0"/>
@@ -56,4 +118,5 @@
     </visual>
   </link>
+  <!-- wheels -->
   <link name='left_wheel'>
     <inertial>
@@ -102,4 +165,5 @@
     </visual>
   </link>
+ <!-- Sensors -->
   <link name='camera'>
     <inertial>
@@ -152,5 +216,5 @@
   </link>
    <joint type="continuous" name="left_wheel_hinge">
-    <origin xyz="0 0.15 0" rpy="0 0 0"/>
+    <origin xyz="0 0.18 0" rpy="0 0 0"/>
     <child link="left_wheel"/>
     <parent link="chassis"/>
@@ -160,5 +224,5 @@
   </joint>
    <joint type="continuous" name="right_wheel_hinge">
-    <origin xyz="0 -0.15 0" rpy="0 0 0"/>
+    <origin xyz="0 -0.18 0" rpy="0 0 0"/>
     <child link="right_wheel"/>
     <parent link="chassis"/>
@@ -168,5 +232,5 @@
   </joint>
    <joint type="fixed" name="camera_joint">
-    <origin xyz="0.2 0 0" rpy="0 0 0"/>
+    <origin xyz="0.2 0 0.055" rpy="0 0 0"/>
     <child link="camera"/>
     <parent link="chassis"/>
@@ -174,5 +238,5 @@
   </joint>
    <joint type="fixed" name="hokuyo_joint">
-    <origin xyz="0.15 0 0.1" rpy="0 0 0"/>
+    <origin xyz="0.15 0 0.26" rpy="0 0 0"/>
     <child link="hokuyo"/>
     <parent link="chassis"/>
