Commit message: none: save latest AMCL parameters to try on cloud

File: Project3/src/my_robot/urdf/my_robot.xacro (robot description, xacro)
@@ -14,5 +14,5 @@
     <inertial>
       <mass value="15.0"/>
-      <origin xyz="0.0 0 0" rpy=" 0 0 0"/>
+      <origin xyz="0 0 0" rpy=" 0 0 0"/>
       <inertia
           ixx="0.1" ixy="0" ixz="0"
@@ -120,4 +120,5 @@
   <!-- wheels -->
   <link name='left_wheel'>
+    <pose>0 0 0.1 0 0 0</pose>
     <inertial>
       <mass value="5.0"/>
@@ -143,4 +144,5 @@
   </link>
   <link name='right_wheel'>
+    <pose>0 0 0.1 0 0 0</pose>
     <inertial>
       <mass value="5.0"/>
